Commit message: Make shelf slots bigger
Former-commit-id: a65b908ae17ea7dc0328a553cfe2162b6babad74

File: reaching_intent/pybullet_models/cabinet/cabinet.urdf (robot description, URDF)
Before this commit: robot cabinet.urdf, 1 links, 0 joints
Links:
- link baseLink: geometry collision mesh filename=cabinet.obj scale=1.5 1.5 1.5; visual mesh filename=cabinet.obj scale=1.5 1.5 1.5
