Commit message: Improved trajectory generation: - Remove joint limits on vel commands - Tune Force Filed controller. Adding distance to goal based force - Touches on velocity limits of the human model - Tuned gains on arm controller tunning - Added IK check mode on controller tunning code
Former-commit-id: a7388720c7fa06b0c4eaa9347376c47e119f68e1

File: reaching_intent/pybullet_models/human_torso/model.urdf (robot description, URDF)
Before this commit: robot human_torso, 24 links, 23 joints
Joints:
- joint l_shoulder_abduction_adduction_joint: limit lower=0.1 upper=3.1415 effort=1000.0 velocity=2.5 -> lower=0.0 upper=3.1415 effort=1000.0 velocity=2.5
- joint r_shoulder_abduction_adduction_joint: limit lower=0.1 upper=3.1415 effort=1000.0 velocity=2.5 -> lower=0.0 upper=3.1415 effort=1000.0 velocity=2.5
- joint torso_frontal_joint: limit lower=-0.2 upper=0.1 effort=10000.0 velocity=0.1 -> lower=-0.1 upper=0.05 effort=10000.0 velocity=0.1
- joint torso_pan_joint: limit lower=-0.2 upper=0.2 effort=10000.0 velocity=1.57 -> lower=-0.2 upper=0.2 effort=10000.0 velocity=0.5
- joint torso_sagital_joint: limit lower=-0.4 upper=0.4 effort=10000.0 velocity=0.1 -> lower=-0.2 upper=0.2 effort=10000.0 velocity=0.1
- joint torso_tilt_joint: limit lower=-0.2 upper=0.2 effort=10000.0 velocity=1.57 -> lower=-0.05 upper=0.2 effort=10000.0 velocity=0.5
