Commit message: Add tranlsational DoF to the human torso
Former-commit-id: ed41efb42b9b65ddd9eba27a991e90adca4ff45f

File: reaching_intent/pybullet_models/human_torso/human_torso.xacro (robot description, xacro)
@@ -24,5 +24,5 @@
         - radial 20
         - ulnar 50
- - generation command: rosrun xacro xacro human_torso.xacro --inorder > model.urdf
+ - generation command: rosrun xacro xacro human_torso.xacro > model.urdf
 -->
 <robot xmlns:xacro="http://www.ros.org/wiki/xacro" name="human_torso">
@@ -356,15 +356,33 @@
     </joint>
 </xacro:macro>
+<xacro:macro name="torso_base" params="prefix base_link translate_joint_type rotate_joint_type *origin">
+    <xacro:property name="torso_forward_limit" value="0.1" />
+    <xacro:property name="torso_backward_limit" value="0.2" />
+    <xacro:property name="torso_left_limit" value="0.4" />
+    <xacro:property name="torso_right_limit" value="0.4" />
+    <xacro:property name="torso_forward_tilt_limit" value="0.2" />
+    <xacro:property name="torso_backward_tilt_limit" value="0.2" />
+    <xacro:property name="torso_pan_limit" value="0.2" />
     <xacro:property name="torso_depth" value="0.2" />
     <xacro:property name="torso_width" value="0.22" />
     <xacro:property name="torso_height" value="0.59" />
     <xacro:property name="torso_joint_type" value="revolute" />
-    <link name="base_link">
-        <inertial>
-           <mass value="0.01" />
-           <origin xyz="0 0 0" rpy="0 0 0"/>
-           <inertia ixx="0.001"  ixy="0"  ixz="0" iyy="0.001" iyz="0" izz="0.001" />
-        </inertial>
-    </link>
+    <!--    Left/right translation-->
+    <link name="torso_sagital_link">
+        <inertial>
+           <mass value="0.01" />
+           <origin xyz="0 0 0" rpy="0 0 0"/>
+           <inertia ixx="0.001"  ixy="0"  ixz="0" iyy="0.001" iyz="0" izz="0.001" />
+        </inertial>
+    </link>
+    <!--    Forward/backward translation-->
+    <link name="torso_frontal_link">
+        <inertial>
+           <mass value="0.01" />
+           <origin xyz="0 0 0" rpy="0 0 0"/>
+           <inertia ixx="0.001"  ixy="0"  ixz="0" iyy="0.001" iyz="0" izz="0.001" />
+        </inertial>
+    </link>
+    <!--    Left/Right rotation-->
     <link name="torso_pan">
         <inertial>
@@ -374,4 +392,5 @@
         </inertial>
     </link>
+    <!--    Forward/backward leaning-->
     <link name="torso">
         <visual>
@@ -394,28 +413,43 @@
         </inertial>
     </link>
-    <joint name="torso_pan_joint" type="${torso_joint_type}">
-        <axis xyz="0 0 1"/>
-        <limit
-            effort="10000.0"
-            lower="-0.32173"
-            upper="0.32173"
-            velocity="1.57"
-        />
-        <origin rpy="0 0 0" xyz="0 0 0"/>
-        <parent link="base_link"/>
-        <child link="torso_pan"/>
-    </joint>
-    <joint name="torso_tilt_joint" type="${torso_joint_type}">
+    <joint name="torso_tilt_joint" type="${rotate_joint_type}">
         <axis xyz="0 1 0"/>
-        <limit
-            effort="10000.0"
-            lower="-0.12173"
-            upper="0.32173"
-            velocity="1.57"
-        />
+        <limit effort="10000.0" lower="-${torso_backward_tilt_limit}" upper="${torso_forward_tilt_limit}" velocity="1.57"/>
         <origin rpy="0 0 0" xyz="0 0 0"/>
         <parent link="torso_pan"/>
         <child link="torso"/>
     </joint>
+    <joint name="torso_pan_joint" type="${rotate_joint_type}">
+        <axis xyz="0 0 1"/>
+        <limit effort="10000.0" lower="-${torso_pan_limit}" upper="${torso_pan_limit}" velocity="1.57"/>
+        <origin rpy="0 0 0" xyz="0 0 0"/>
+        <parent link="torso_sagital_link"/>
+        <child link="torso_pan"/>
+    </joint>
+    <joint name="torso_sagital_joint" type="${translate_joint_type}">
+        <axis xyz="0 1 0"/>
+        <limit effort="10000.0" lower="-${torso_right_limit}" upper="${torso_left_limit}" velocity="0.1"/>
+        <origin rpy="0 0 0" xyz="0 0 0"/>
+        <parent link="torso_frontal_link"/>
+        <child link="torso_sagital_link"/>
+    </joint>
+    <joint name="torso_frontal_joint" type="${translate_joint_type}">
+        <axis xyz="1 0 0"/>
+        <limit effort="10000.0" lower="-${torso_backward_limit}" upper="${torso_forward_limit}" velocity="0.1"/>
+        <xacro:insert_block name="origin"/>
+        <parent link="${base_link}"/>
+        <child link="torso_frontal_link"/>
+    </joint>
+</xacro:macro>
+    <link name="base_link">
+        <inertial>
+           <mass value="0.01" />
+           <origin xyz="0 0 0" rpy="0 0 0"/>
+           <inertia ixx="0.001"  ixy="0"  ixz="0" iyy="0.001" iyz="0" izz="0.001" />
+        </inertial>
+    </link>
+    <xacro:torso_base prefix="" base_link="base_link" rotate_joint_type="revolute" translate_joint_type="prismatic">
+        <origin xyz=" 0 0 0" rpy="0 0 0" />
+    </xacro:torso_base>
     <xacro:human_arm prefix="l_" base_link="torso" reflect="1" joint_type="revolute">
         <origin xyz=" 0 0.10988 0.4938" rpy="0 0 0" />

File: reaching_intent/pybullet_models/human_torso/model.urdf (robot description, URDF)
Before this commit: robot human_torso, 22 links, 21 joints
Links:
- added link torso_frontal_link, mass 0.01
- added link torso_sagital_link, mass 0.01
Joints:
- added joint torso_frontal_joint: type prismatic, parent base_link, child torso_frontal_link, origin xyz= 0 0 0 rpy=0 0 0, axis 1 0 0, limit lower=-0.2 upper=0.1 effort=10000.0 velocity=0.1
- added joint torso_sagital_joint: type prismatic, parent torso_frontal_link, child torso_sagital_link, origin xyz=0 0 0 rpy=0 0 0, axis 0 1 0, limit lower=-0.4 upper=0.4 effort=10000.0 velocity=0.1
- joint torso_pan_joint: limit lower=-0.32173 upper=0.32173 effort=10000.0 velocity=1.57 -> lower=-0.2 upper=0.2 effort=10000.0 velocity=1.57; parent base_link -> torso_sagital_link
- joint torso_tilt_joint: limit lower=-0.12173 upper=0.32173 effort=10000.0 velocity=1.57 -> lower=-0.2 upper=0.2 effort=10000.0 velocity=1.57

Commit message: fixup with previous
Former-commit-id: 4f3a8c6e65a4bdf37ab8322b7e346b2816dabbae

File: reaching_intent/pybullet_models/human_torso/human_torso.xacro (robot description, xacro)
@@ -129,5 +129,5 @@
     <xacro:property name="palm_depth" value="0.11" />
     <xacro:property name="shoulder_abduction_limit" value="3.1415" />
-    <xacro:property name="shoulder_adduction_limit" value="0.1" />
+    <xacro:property name="shoulder_adduction_limit" value="0.0" />
     <xacro:property name="shoulder_abduction_adduction_effort" value="1000.0" />
     <xacro:property name="shoulder_abduction_adduction_velocity" value="2.5" />
@@ -357,10 +357,10 @@
 </xacro:macro>
 <xacro:macro name="torso_base" params="prefix base_link translate_joint_type rotate_joint_type *origin">
-    <xacro:property name="torso_forward_limit" value="0.1" />
-    <xacro:property name="torso_backward_limit" value="0.2" />
-    <xacro:property name="torso_left_limit" value="0.4" />
-    <xacro:property name="torso_right_limit" value="0.4" />
+    <xacro:property name="torso_forward_limit" value="0.05" />
+    <xacro:property name="torso_backward_limit" value="0.1" />
+    <xacro:property name="torso_left_limit" value="0.2" />
+    <xacro:property name="torso_right_limit" value="0.2" />
     <xacro:property name="torso_forward_tilt_limit" value="0.2" />
-    <xacro:property name="torso_backward_tilt_limit" value="0.2" />
+    <xacro:property name="torso_backward_tilt_limit" value="0.05" />
     <xacro:property name="torso_pan_limit" value="0.2" />
     <xacro:property name="torso_depth" value="0.2" />
@@ -415,5 +415,5 @@
     <joint name="torso_tilt_joint" type="${rotate_joint_type}">
         <axis xyz="0 1 0"/>
-        <limit effort="10000.0" lower="-${torso_backward_tilt_limit}" upper="${torso_forward_tilt_limit}" velocity="1.57"/>
+        <limit effort="10000.0" lower="-${torso_backward_tilt_limit}" upper="${torso_forward_tilt_limit}" velocity="0.5"/>
         <origin rpy="0 0 0" xyz="0 0 0"/>
         <parent link="torso_pan"/>
@@ -422,5 +422,5 @@
     <joint name="torso_pan_joint" type="${rotate_joint_type}">
         <axis xyz="0 0 1"/>
-        <limit effort="10000.0" lower="-${torso_pan_limit}" upper="${torso_pan_limit}" velocity="1.57"/>
+        <limit effort="10000.0" lower="-${torso_pan_limit}" upper="${torso_pan_limit}" velocity="0.5"/>
         <origin rpy="0 0 0" xyz="0 0 0"/>
         <parent link="torso_sagital_link"/>
@@ -429,5 +429,5 @@
     <joint name="torso_sagital_joint" type="${translate_joint_type}">
         <axis xyz="0 1 0"/>
-        <limit effort="10000.0" lower="-${torso_right_limit}" upper="${torso_left_limit}" velocity="0.1"/>
+        <limit effort="10000.0" lower="-${torso_right_limit}" upper="${torso_left_limit}" velocity="0.2"/>
         <origin rpy="0 0 0" xyz="0 0 0"/>
         <parent link="torso_frontal_link"/>
@@ -436,5 +436,5 @@
     <joint name="torso_frontal_joint" type="${translate_joint_type}">
         <axis xyz="1 0 0"/>
-        <limit effort="10000.0" lower="-${torso_backward_limit}" upper="${torso_forward_limit}" velocity="0.1"/>
+        <limit effort="10000.0" lower="-${torso_backward_limit}" upper="${torso_forward_limit}" velocity="0.2"/>
         <xacro:insert_block name="origin"/>
         <parent link="${base_link}"/>
